File: KiCad/KiCad.kicad_sch (KiCad schematic)
At the start: 50 parts, among them J1 DC-IN, J2 TYPE-C, J3 Conn_01x03_Pin, J4 Conn_01x03_Pin, J5 Conn_01x03_Pin, J6 Conn_01x03_Pin, Q1 IRF3708, SW1 reset, SW2 start, U1 ESP32-WROOM-32E, U2 MP1584EN, U3 CH340C, U4 RT9013-33GB, U5 DM-OLED096-636, U6 INA232AIDDFR, U7 MIC4420YM, U8 LM358

Commit message: 基礎定速與外設完成
Parts:
- added D4: SS14, Diode_SMD:D_SMA, symbol Diode:SS14
Connections:
- net +5V: now also D4.1 (K); no longer J2.A4_B9 (VBUS), J2.B4_A9 (VBUS)
- new net VBUS: D4.2 (A), J2.A4_B9 (VBUS), J2.B4_A9 (VBUS)
Changed lines of the file:
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@@
 	(wire
 		(pts
-			(xy 224.79 124.46) (xy 222.25 124.46)
-		)
-		(stroke
-			(width 0)
-			(type default)
-		)
-	)
-	(wire
-		(pts
 			(xy 115.57 109.22) (xy 115.57 106.68)
 		)
@@
 	(wire
 		(pts
+			(xy 232.41 124.46) (xy 229.87 124.46)
+		)
+		(stroke
+			(width 0)
+			(type default)
+		)
+	)
+	(wire
+		(pts
 			(xy 273.05 80.01) (xy 273.05 74.93)
 		)
@@
 	(wire
 		(pts
+			(xy 232.41 120.65) (xy 232.41 124.46)
+		)
+		(stroke
+			(width 0)
+			(type default)
+		)
+	)
+	(wire
+		(pts
 			(xy 90.17 160.02) (xy 90.17 165.1)
 		)
@@
 	)
 	(symbol
+		(lib_id "Diode:SS14")
+		(at 226.06 124.46 180)
+		(unit 1)
+		(exclude_from_sim no)
+		(in_bom yes)
+		(on_board yes)
+		(dnp no)
+		(fields_autoplaced yes)
+		(property "Reference" "D4"
+			(at 226.3775 118.11 0)
+			(effects
+				(font
+					(size 1.27 1.27)
+				)
+			)
+		)
+		(property "Value" "SS14"
+			(at 226.3775 120.65 0)
+			(effects
+				(font
+					(size 1.27 1.27)
+				)
+			)
+		)
+		(property "Footprint" "Diode_SMD:D_SMA"
+			(at 226.06 120.015 0)
+			(effects
+				(font
+					(size 1.27 1.27)
+				)
+				(hide yes)
+			)
+		)
+		(property "Datasheet" "https://www.vishay.com/docs/88746/ss12.pdf"
+			(at 226.06 124.46 0)
+			(effects
+				(font
+					(size 1.27 1.27)
+				)
+				(hide yes)
+			)
+		)
+		(property "Description" "40V 1A Schottky Diode, SMA"
+			(at 226.06 124.46 0)
+			(effects
+				(font
+					(size 1.27 1.27)
+				)
+				(hide yes)
+			)
+		)
+		(pin "2"
+		)
+		(pin "1"
+		)
+		(instances
+			(project "KiCad"
+				(path "/8145d5a2-4aff-47fb-b6a2-0059c8017b6c"
+					(reference "D4")
+					(unit 1)
+				)
+			)
+		)
+	)
+	(symbol
 		(lib_id "power:GND")
 		(at 57.15 93.98 0)
@@
 	(symbol
 		(lib_id "power:+5V")
-		(at 224.79 124.46 0)
+		(at 232.41 120.65 0)
 		(unit 1)
 		(exclude_from_sim no)
@@
 		(fields_autoplaced yes)
 		(property "Reference" "#PWR017"
-			(at 224.79 128.27 0)
+			(at 232.41 124.46 0)
 			(effects
 				(font
@@
 		)
 		(property "Value" "+5V"
-			(at 224.79 119.38 0)
+			(at 232.41 115.57 0)
 			(effects
 				(font
@@
 		)
 		(property "Footprint" ""
-			(at 224.79 124.46 0)
+			(at 232.41 120.65 0)
 			(effects
 				(font
@@
 		)
 		(property "Datasheet" ""
-			(at 224.79 124.46 0)
+			(at 232.41 120.65 0)
 			(effects
 				(font
@@
 		)
 		(property "Description" "Power symbol creates a global label with name \"+5V\""
-			(at 224.79 124.46 0)
+			(at 232.41 120.65 0)
 			(effects
 				(font
