File: KiCad/KiCad.kicad_pcb (KiCad board)
At the start: 2 copper layers, 100 x 46.3 mm, 50 parts, among them J1 DC-IN, J2 TYPE-C, J3 Conn_01x03_Pin, J4 Conn_01x03_Pin, J5 Conn_01x03_Pin, J6 Conn_01x03_Pin, Q1 IRF3708, SW1 reset, SW2 start, U1 ESP32-WROOM-32E, U2 MP1584EN, U3 CH340C, U4 RT9013-33GB, U5 DM-OLED096-636, U6 INA232AIDDFR, U7 MIC4420YM, U8 LM358

Commit message: 基礎定速與外設完成
Parts:
- added D4: SS14, Diode_SMD:D_SMA, F.Cu at (224.0, 86.8)
Connections:
- J2 pad A4_B9: +5V -> VBUS
- J2 pad B4_A9: +5V -> VBUS
Routing:
- net VBUS: track 0.00 -> 18.7 mm
- net +5V: track 148.5 -> 139.5 mm, vias 5 -> 6
